File: HE60/HE60.kicad_pcb (KiCad board)
At the start: 2 copper layers, 284.7 x 94.2 mm, 267 parts, among them J1 TYPE-C-31-M-12, J2 JST_SH, J3 TC2030, SW1 TS-1187A-B-A-B, SW2 TS-1187A-B-A-B, U1 STM32F446RET6, U2 USBLC6-2SC6, U3 TLV75733PDBVR, U4 TLV75733PDBVR, Y1 X322516MLB4SI

Commit message: :sparkles: add logo
Routing:
- net GND: vias 1246 -> 1783
