File: HE60/HE60.kicad_pcb (KiCad board)
At the start: 2 copper layers, 284.7 x 94.2 mm, 267 parts, among them J1 TYPE-C-31-M-12, J2 JST_SH, J3 TC2030, SW1 TS-1187A-B-A-B, SW2 TS-1187A-B-A-B, U1 STM32F446RET6, U2 USBLC6-2SC6, U3 TLV75733PDBVR, U4 TLV75733PDBVR, Y1 X322516MLB4SI

Commit message: :art: tidy up some traces
Routing:
- net ADC_IN_4: track 74.3 -> 71.4 mm
- net ADC_IN_2: track 73.2 -> 71.5 mm
- net SWO: track 26.1 -> 27.8 mm
- net ADC_IN_3: track 64.8 -> 63.3 mm
- net MUX_SELECT_0: track 336.4 -> 337.0 mm
- net ADC_IN_1: track 56.3 -> 55.8 mm
- net GND: vias 1783 -> 1801

Commit message: :art: move buttons further from the switch
Parts:
- moved R4 6.54 mm to (36.1, 67.8), turned to 180 degrees
- moved SW1 2.21 mm to (40.1, 56.8)
- moved SW2 2.21 mm to (40.1, 64.8)
Routing:
- net +3.3VA: track 1764.8 -> 1756.7 mm, vias 27 -> 26
- net +3.3V: track 170.4 -> 168.1 mm
- net NRST: track 58.7 -> 56.7 mm
- net BOOT0: track 42.8 -> 42.1 mm
- net GND: vias 1801 -> 1799

Commit message: :sparkles: update PCB & plate
Parts:
- TH1, TH2: moved to B.Cu
- moved H4 152.4 mm to (66.2, 37.6)
- moved H3 138.2 mm to (280.5, 23.3)
- moved H6 114.7 mm to (142.3, 75.7)
- moved H7 114.7 mm to (28.1, 85.2)
- moved C71 87.8 mm to (162.6, 40.6)
- moved H2 78.5 mm to (142.3, 18.5)
- moved C72 76.2 mm to (76.8, 59.6)
- moved H5 63.5 mm to (218.6, 37.6)
- moved C75 42.9 mm to (114.9, 78.7)
- moved C76 42.9 mm to (157.8, 78.7)
- moved AM8 42.9 mm to (118.5, 75.7)
- moved AM9 42.9 mm to (161.4, 75.7)
- moved R4 34.0 mm to (43.4, 34.6), turned to -90 degrees
- moved SW2 28.1 mm to (47.1, 37.6)
- moved SW1 23.6 mm to (53.9, 37.6)
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Connections:
- AM8 pad 1: HE50 -> HE47
- AM8 pad 12: HE65 -> HE61
- AM8 pad 13: HE66 -> HE62
- AM8 pad 14: HE67 -> HE63
- AM8 pad 15: HE54 -> HE64
- AM8 pad 2: HE51 -> unconnected-(AM8-X6-Pad2)
- AM8 pad 4: HE52 -> HE48
- AM8 pad 5: HE53 -> HE49
- AM9 pad 1: HE47 -> HE50
- AM9 pad 12: HE61 -> HE65
- AM9 pad 13: HE62 -> HE66
- AM9 pad 14: HE63 -> HE67
- AM9 pad 15: HE64 -> HE54
- AM9 pad 2: unconnected-(AM9-X6-Pad2) -> HE51
- AM9 pad 4: HE48 -> HE52
- AM9 pad 5: HE49 -> HE53
- OP2 pad 10: unconnected-(OP2C-+-Pad10) -> GND
- OP2 pad 5: unconnected-(OP2B-+-Pad5) -> GND
- OP2 pad 6: unconnected-(OP2B---Pad6) -> Net-(OP2B--)
- OP2 pad 7: unconnected-(OP2-Pad7) -> Net-(OP2B--)
- OP2 pad 8: unconnected-(OP2-Pad8) -> Net-(OP2C--)
- OP2 pad 9: unconnected-(OP2C---Pad9) -> Net-(OP2C--)
- OP3 pad 1: ADC_IN_8 -> ADC_IN_9
- OP3 pad 10: MUX_OUT_9 -> MUX_OUT_8
- OP3 pad 2: ADC_IN_8 -> ADC_IN_9
- OP3 pad 3: MUX_OUT_8 -> MUX_OUT_9
- OP3 pad 5: unconnected-(OP3B-+-Pad5) -> GND
- OP3 pad 6: unconnected-(OP3B---Pad6) -> Net-(OP3B--)
- OP3 pad 7: unconnected-(OP3-Pad7) -> Net-(OP3B--)
- OP3 pad 8: ADC_IN_9 -> ADC_IN_8
- OP3 pad 9: ADC_IN_9 -> ADC_IN_8
- U1 pad 26: ADC_IN_9 -> ADC_IN_8
- U1 pad 27: ADC_IN_8 -> ADC_IN_9
Routing:
- net +3.3VA: track 1756.7 -> 1705.5 mm
- net MUX_OUT_9: track 74.1 -> 119.3 mm
- net MUX_OUT_8: track 116.0 -> 74.9 mm
- net +3.3V: track 168.1 -> 187.7 mm
- net BOOT0: track 42.1 -> 24.2 mm, vias 4 -> 0
- net NRST: track 56.7 -> 74.0 mm, vias 3 -> 2
- net GND: track 232.0 -> 219.7 mm, vias 1799 -> 1821
- net ADC_IN_8: track 50.0 -> 38.5 mm
- net ADC_IN_9: track 39.9 -> 47.9 mm
- net SWCLK: track 29.5 -> 37.3 mm
- net SWO: track 27.8 -> 34.9 mm
- net MUX_SELECT_0: track 337.0 -> 331.4 mm
- net HE28: track 73.7 -> 79.1 mm
- net MUX_SELECT_1: track 335.3 -> 330.2 mm
- net USB_D-: track 64.5 -> 69.5 mm
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- removed copper zone on B.Cu, net +3.3V
- removed copper zone on B.Cu, net +3.3VA

Commit message: :fire: remove op amp & update PCB
Parts:
- removed C93, C94, C95: 2.2u, Capacitor_SMD:C_0603_1608Metric
- removed OP1, OP2, OP3: GS8094-SR, Package_SO:SOIC-14_3.9x8.7mm_P1.27mm
- removed U4: TLV75733PDBVR, Package_TO_SOT_SMD:SOT-23-5
- added FB1: 100R@100MHz, Inductor_SMD:L_0805_2012Metric, B.Cu at (13.1, 19.5)
- AM1, AM2, AM3, AM4, AM5, AM6, AM7, AM8, AM9: value TMUX1308PWR -> SN74LV4051A
- C77, C78: value 100n -> 2.2u; footprint Capacitor_SMD:C_0402_1005Metric -> Capacitor_SMD:C_0603_1608Metric
- C79, C80: value 100n -> 1u; footprint Capacitor_SMD:C_0402_1005Metric -> Capacitor_SMD:C_0603_1608Metric
- C85: value 10u -> 100n; footprint Capacitor_SMD:C_0603_1608Metric -> Capacitor_SMD:C_0402_1005Metric
- C86: value 100n -> 10u; footprint Capacitor_SMD:C_0402_1005Metric -> Capacitor_SMD:C_0603_1608Metric
- C87: value 1u -> 100n; footprint Capacitor_SMD:C_0603_1608Metric -> Capacitor_SMD:C_0402_1005Metric
- C88: value 4.7u -> 1u
- C89: value 10p -> 100n
- C90: value 10p -> 4.7u; footprint Capacitor_SMD:C_0402_1005Metric -> Capacitor_SMD:C_0603_1608Metric
- C91: value 100n -> 10p
- C92: value 2.2u -> 10p; footprint Capacitor_SMD:C_0603_1608Metric -> Capacitor_SMD:C_0402_1005Metric
- F1: value BSMD1206-100-16V -> BSMD0805-050-24V; footprint Fuse:Fuse_1206_3216Metric -> Fuse:Fuse_0805_2012Metric
- H1, H2, H3, H4, H5, H6, H7, H8: footprint HE60:SpacerHole -> MountingHole:MountingHole_2.2mm_M2_Pad
- HE1, HE10, HE11, HE12, HE13, HE14, HE15, HE16, HE17, HE18, HE19, HE2, HE20, HE21, HE22, HE23, HE24, HE25, HE26, HE27, HE28, HE29, HE3, HE30, HE31, HE32, HE33, HE34, HE35, HE36, HE37, HE38, HE39, HE4, HE40, HE41, HE42, HE43, HE44, HE45, HE46, HE47, HE48, HE49, HE5, HE50, HE51, HE52, HE53, HE54, HE55, HE56, HE57, HE58, HE59, HE6, HE60, HE61, HE62, HE63, HE64, HE65, HE66, HE67, HE7, HE8, HE9: value GH39F -> OH49E-S
- MX57: value 1.5 -> 1.5U
- R1: value 10k -> 5.1k
- R3: value 5.1k -> 10k
- U1: value STM32F446RET6 -> USBLC6-2SC6; footprint Package_QFP:LQFP-64_10x10mm_P0.5mm -> Package_TO_SOT_SMD:SOT-23-6
- U2: value USBLC6-2SC6 -> TLV75733PDBV; footprint Package_TO_SOT_SMD:SOT-23-6 -> Package_TO_SOT_SMD:SOT-23-5
- U3: value TLV75733PDBVR -> STM32F446RET6; footprint Package_TO_SOT_SMD:SOT-23-5 -> Package_QFP:LQFP-64_10x10mm_P0.5mm
- moved C79 70.0 mm to (15.1, 17.7), turned to 90 degrees
- moved R3 62.3 mm to (21.7, 71.0), turned to 0 degrees
- moved C78 53.5 mm to (29.1, 18.1), turned to -90 degrees
- moved SW1 47.4 mm to (25.7, 75.7)
- moved SW2 47.2 mm to (19.3, 75.7), turned to 90 degrees
- moved C77 46.4 mm to (35.5, 17.9), turned to -90 degrees
- moved R1 42.6 mm to (16.4, 9.00)
- moved C80 24.5 mm to (15.1, 21.3), turned to -90 degrees
- moved U1 23.9 mm to (40.7, 20.1)
- moved R4 21.7 mm to (27.2, 49.0)
- moved U3 20.7 mm to (29.2, 41.0)
- moved C92 19.9 mm to (39.2, 39.8), turned to 90 degrees
- moved C86 17.9 mm to (20.0, 36.4), turned to -90 degrees
- moved C88 17.0 mm to (39.2, 42.6), turned to 0 degrees
- moved C90 16.5 mm to (24.6, 50.2), turned to 180 degrees
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Connections:
- AM3 pad 14: unconnected-(AM3-X1-Pad14) -> GND
- AM3 pad 15: unconnected-(AM3-X2-Pad15) -> GND
- AM5 pad 15: unconnected-(AM5-X2-Pad15) -> GND
- AM5 pad 5: unconnected-(AM5-X5-Pad5) -> GND
- AM8 pad 2: unconnected-(AM8-X6-Pad2) -> GND
- C77 pad 1: +3.3VA -> +5V
- C78 pad 1: +3.3VA -> +3.3V
- C79 pad 1: +3.3VA -> +3.3V
- C80 pad 1: +3.3V -> +3.3VA
- C86 pad 1: +3.3VA -> +3.3V
- C88 pad 1: Net-(U1-VCAP_1) -> +3.3VA
- C89 pad 1: /RCC_OSC_IN -> GND
- C89 pad 2: GND -> NRST
- C90 pad 1: /RCC_OSC_OUT -> Net-(U3-VCAP_1)
- C91 pad 1: GND -> /RCC_OSC_IN
- C91 pad 2: NRST -> GND
- C92 pad 1: +5V -> /RCC_OSC_OUT
- J2 pad MP: (no net) -> unconnected-(J2-MountPin-PadMP)
- R1 pad 1: /BOOT1 -> Net-(J1-CC1)
- R2 pad 1: Net-(J1-CC1) -> GND
- R2 pad 2: GND -> Net-(J1-CC2)
- R3 pad 1: GND -> BOOT0
- R3 pad 2: Net-(J1-CC2) -> GND
- R4 pad 1: BOOT0 -> /BOOT1
- U1 pad 1: +3.3V -> USB_PLUG_D-
- U1 pad 2: MUX_SELECT_0 -> GND
- U1 pad 3: MUX_SELECT_1 -> USB_PLUG_D+
- U1 pad 4: MUX_SELECT_2 -> USB_D+
- U1 pad 5: /RCC_OSC_IN -> +5V
- U1 pad 6: /RCC_OSC_OUT -> USB_D-
- U2 pad 1: USB_PLUG_D- -> +5V
- U2 pad 3: USB_PLUG_D+ -> +5V
- U2 pad 4: USB_D+ -> unconnected-(U2-NC-Pad4)
- U2 pad 5: +5V -> +3.3V
- U3 pad 1: +5V -> +3.3V
- U3 pad 2: GND -> MUX_SELECT_0
- U3 pad 3: +5V -> MUX_SELECT_1
- U3 pad 4: unconnected-(U3-NC-Pad4) -> MUX_SELECT_2
- U3 pad 5: +3.3V -> /RCC_OSC_IN
Routing:
- net ADC_IN_4: track 68.0 -> 0.00 mm, vias 2 -> 0
- net ADC_IN_2: track 67.2 -> 0.00 mm, vias 2 -> 0
- net MUX_OUT_2: track 101.3 -> 167.4 mm
- net MUX_OUT_1: track 45.2 -> 106.3 mm
- net MUX_OUT_3: track 17.5 -> 76.9 mm, vias 0 -> 2
- net ADC_IN_3: track 59.1 -> 0.00 mm, vias 2 -> 0
- net MUX_OUT_4: track 95.3 -> 152.5 mm, vias 0 -> 2
- net ADC_IN_1: track 57.0 -> 0.00 mm, vias 2 -> 0
- net ADC_IN_9: track 47.9 -> 0.00 mm, vias 2 -> 0
- net ADC_IN_7: track 46.7 -> 0.00 mm, vias 2 -> 0
- net GND: track 219.7 -> 174.2 mm, vias 1821 -> 1941
- net ADC_IN_6: track 45.2 -> 0.00 mm
- net ADC_IN_5: track 44.4 -> 0.00 mm
- net BOOT0: track 24.2 -> 66.7 mm, vias 0 -> 2
- net MUX_OUT_7: track 28.6 -> 68.0 mm, vias 0 -> 2
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- added copper zone on B.Cu, net +3.3V
Other:
- board text added: "BOOT"
- board text removed: "BOOT0"
