File: HE60/HE60.kicad_pcb (KiCad board)
At the start: 2 copper layers, 284.7 x 94.2 mm, 261 parts, among them J1 TYPE-C-31-M-12, J2 JST_SH, J3 TC2030, SW1 TS-1187A-B-A-B, SW2 TS-1187A-B-A-B, U1 USBLC6-2SC6, U2 TLV75733PDBV, U3 STM32F446RET6, Y1 X322516MLB4SI

Commit message: :sparkles: separate voltage supplier for MCU
Parts:
- removed C79, C80: 1u, Capacitor_SMD:C_0603_1608Metric
- removed FB1: 100R@100MHz, Inductor_SMD:L_0805_2012Metric
- added C93: 1u, Capacitor_SMD:C_0603_1608Metric, B.Cu at (37.3, 17.3)
- added C94: 1u, Capacitor_SMD:C_0603_1608Metric, B.Cu at (34.3, 20.7)
- added U4: XC6206P332MR-G, Package_TO_SOT_SMD:SOT-23-3, B.Cu at (34.5, 17.5)
- moved C77 6.87 mm to (28.7, 16.9)
- moved C78 6.87 mm to (22.3, 17.1)
- moved U2 6.87 mm to (25.5, 17.3)
Connections:
- C78 pad 1: +3.3V -> +3.3VA
- U2 pad 5: +3.3V -> +3.3VA
Routing:
- net +3.3V: track 197.3 -> 193.4 mm
- net USB_D-: track 66.1 -> 68.7 mm
- net GND: track 174.2 -> 172.2 mm, vias 1941 -> 1945
- net USB_D+: track 64.2 -> 66.2 mm
- net +3.3VA: track 1672.9 -> 1674.6 mm
- added copper zone on B.Cu, net +3.3VA

Commit message: :bug: fix escape key noise
Parts:
- moved R3 1.60 mm to (20.1, 71.1)
- moved SW1 1.56 mm to (24.1, 75.7)
- moved SW2 1.56 mm to (17.7, 75.7)
- moved C78 1.09 mm to (21.4, 17.8)
- moved U2 1.09 mm to (24.6, 18.0)
- moved C89 1.00 mm to (46.0, 42.2)
- moved U4 0.97 mm to (33.6, 18.0)
- moved C93 0.97 mm to (36.5, 17.8)
- moved C94 0.97 mm to (33.5, 21.2)
- moved C77 0.94 mm to (28.1, 17.6)
- moved C88 0.60 mm to (39.2, 43.2)
- moved C87 0.20 mm to (36.8, 42.6)
- moved C92 0.20 mm to (39.2, 40.0)
- moved Y1 0.20 mm to (41.8, 39.0)
- moved R1 0.20 mm to (16.4, 9.20)
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Connections:
- AM1 pad 12: HE4 -> GND
- AM1 pad 13: HE3 -> HE4
- AM1 pad 14: HE2 -> HE3
- AM1 pad 15: HE1 -> HE2
- AM3 pad 1: HE17 -> HE20
- AM3 pad 12: HE22 -> HE19
- AM3 pad 13: HE21 -> HE18
- AM3 pad 14: GND -> HE17
- AM3 pad 15: GND -> HE1
- AM3 pad 2: HE18 -> GND
- AM3 pad 4: HE19 -> HE21
- AM3 pad 5: HE20 -> HE22
Routing:
- net GND: track 172.2 -> 187.9 mm, vias 1945 -> 1897
- net HE1: track 98.7 -> 109.0 mm
- net HE17: track 76.2 -> 83.0 mm
- net HE18: track 53.5 -> 59.8 mm
- net +3.3VA: track 1674.6 -> 1669.4 mm, vias 22 -> 20
- net HE21: track 17.5 -> 13.5 mm
- net HE19: track 35.7 -> 38.9 mm
- net HE20: track 17.4 -> 14.3 mm
- net HE22: track 34.4 -> 31.9 mm
- net BOOT0: track 66.7 -> 64.5 mm
- net MUX_OUT_1: track 106.3 -> 108.4 mm
- net HE28: track 78.0 -> 76.1 mm
- net MUX_OUT_2: track 167.4 -> 169.2 mm
- net MUX_SELECT_1: track 331.7 -> 333.0 mm
- net MUX_SELECT_2: track 333.1 -> 334.4 mm
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
Commit message: :bug: fix spacebar standoff position
Parts:
- moved H6 41.6 mm to (182.8, 85.2)
Routing:
- net GND: vias 1897 -> 1899
